File: avt953.brd (EAGLE design)
At the start: 100 x 80 mm, 51 parts, among them CON3 RJ45-6L2-B, CON4A MKDS_5/3-6,35, CON4B MKDS_5/3-6,35, CON4C MKDS_5/3-6,35, CON4D MKDS_5/3-6,35, X1 20MHz, X2 20MHz

Commit message: Poprawiono krytyczny błąd. Trzy elementy SMD na warstwie bottom nachodziły na siebie.
Parts:
- moved C8 4.45 mm to (21.7, 46.4)
- moved C10 4.32 mm to (20.8, 30.2)
Routing:
- net N$7: track 15.5 -> 24.1 mm
- net N$6: track 8.36 -> 13.2 mm
- net N$5: track 6.14 -> 10.6 mm
- net N$3: track 4.08 -> 7.94 mm
- net N$4: track 4.29 -> 7.88 mm
- net N$2: track 70.6 -> 73.3 mm
- net N$1: track 19.6 -> 20.5 mm
- net VCC: track 350.2 -> 349.4 mm
- net GND: vias 26 -> 27
